Commit message: Added linear actuator cylinder for visualization

File: src/lx_autonomy/src/lx_packages/lx_description/urdf/lunarx.urdf.xacro (robot description, xacro)
@@ -90,4 +90,20 @@
         <child link="lift_assembly_link" />
     </joint>
+    <link name="lin_act_cylinder_link">
+        <visual>
+            <origin xyz="0 0 0" rpy="0 0 0" />
+            <geometry>
+                <cylinder length="0.1" radius="0.02"/>
+            </geometry>
+            <material name="lin_act_cylinder_black">
+                <color rgba="0 0 0 1"/>
+            </material>
+        </visual>
+    </link>
+    <joint name="lin_act_cylinder_joint" type="fixed">
+        <origin xyz="0 -0.035 -0.055" rpy="0 0 0" />
+        <parent link="lin_act_upper_link" />
+        <child link="lin_act_cylinder_link" />
+    </joint>
     <!-- Electronics plate -->
     <link name="electronics_plate_link">

Commit message: rtabmap VO inaccuracy tested

File: src/lx_autonomy/src/lx_packages/lx_description/urdf/lunarx.urdf.xacro (robot description, xacro)
@@ -171,5 +171,5 @@
     <link name="vectornav"/>
     <joint name="vectornav_joint" type="fixed">
-        <origin xyz="0.17 0 0.52" rpy="1.5707 0 0" />
+        <origin xyz="0.17 0 0.52" rpy="0 0 1.5707" />
         <parent link="base_footprint" />
         <child link="vectornav" />
@@ -178,5 +178,5 @@
     <link name="total_station_prism"/>
     <joint name="total_station_prism_joint" type="fixed">
-        <origin xyz="0.27 0.19 0.8" rpy="1.5707 0 0" />
+        <origin xyz="0.27 0.19 0.8" rpy="0 0 1.5707" />
         <parent link="base_footprint" />
         <child link="total_station_prism" />

Commit message: added imu orientation to TS to fix calib issue

File: src/lx_autonomy/src/lx_packages/lx_description/urdf/lunarx.urdf.xacro (robot description, xacro)
@@ -169,16 +169,16 @@
     </joint>
     <!-- IMU -->
-    <link name="vectornav"/>
+    <!-- <link name="vectornav"/>
     <joint name="vectornav_joint" type="fixed">
         <origin xyz="0.17 0 0.52" rpy="1.5707 0 0" />
         <parent link="base_footprint" />
         <child link="vectornav" />
-    </joint>
+    </joint> -->
     <!-- Total Station Prism -->
-    <link name="total_station_prism"/>
+    <!-- <link name="total_station_prism"/>
     <joint name="total_station_prism_joint" type="fixed">
         <origin xyz="0.27 0.19 0.8" rpy="1.5707 0 0" />
         <parent link="base_footprint" />
         <child link="total_station_prism" />
-    </joint>
+    </joint> -->
 </robot>

Commit message: Restructured localization fix and prepared for integration

File: src/lx_autonomy/src/lx_packages/lx_description/urdf/lunarx.urdf.xacro (robot description, xacro)
@@ -169,16 +169,16 @@
     </joint>
     <!-- IMU -->
-    <!-- <link name="vectornav"/>
+    <link name="vectornav"/>
     <joint name="vectornav_joint" type="fixed">
         <origin xyz="0.17 0 0.52" rpy="1.5707 0 0" />
         <parent link="base_footprint" />
         <child link="vectornav" />
-    </joint> -->
+    </joint>
     <!-- Total Station Prism -->
-    <!-- <link name="total_station_prism"/>
+    <link name="total_station_prism"/>
     <joint name="total_station_prism_joint" type="fixed">
-        <origin xyz="0.27 0.19 0.8" rpy="1.5707 0 0" />
+        <origin xyz="0.27 0.19 0.8" rpy="0 0 0" />
         <parent link="base_footprint" />
         <child link="total_station_prism" />
-    </joint> -->
+    </joint>
 </robot>

Commit message: fixed static transforms and handled edge cases

File: src/lx_autonomy/src/lx_packages/lx_description/urdf/lunarx.urdf.xacro (robot description, xacro)
@@ -171,5 +171,5 @@
     <link name="vectornav"/>
     <joint name="vectornav_joint" type="fixed">
-        <origin xyz="0.17 0 0.52" rpy="1.5707 0 0" />
+        <origin xyz="0.17 0 0.52" rpy="0 0 1.5707" />
         <parent link="base_footprint" />
         <child link="vectornav" />

Commit message: hot fixes 2

File: src/lx_autonomy/src/lx_packages/lx_description/urdf/lunarx.urdf.xacro (robot description, xacro)
@@ -178,5 +178,5 @@
     <link name="total_station_prism"/>
     <joint name="total_station_prism_joint" type="fixed">
-        <origin xyz="0.27 0.19 0.8" rpy="0 0 0" />
+        <origin xyz="0.2625 0.18 0.8" rpy="0 0 0" />
         <parent link="base_footprint" />
         <child link="total_station_prism" />

Commit message: integration tested

File: src/lx_autonomy/src/lx_packages/lx_description/urdf/lunarx.urdf.xacro (robot description, xacro)
@@ -142,5 +142,8 @@
     <link name="camera_link"/>
     <joint type="fixed" name="camera_link_joint">
-        <origin xyz="0.27 0.21 0.7" rpy="0 0.65 -0.16" />
+        <!-- old values  -->
+        <!-- <origin xyz="0.27 0.21 0.7" rpy="0 0.65 -0.16" /> -->
+        <!-- New values -->
+        <origin xyz="0.285 0.21 0.77" rpy="0.0 0.64 -0.14" />
         <parent link="base_footprint" />
         <child link="camera_link" />

Commit message: integration tested curved berm

File: src/lx_autonomy/src/lx_packages/lx_description/urdf/lunarx.urdf.xacro (robot description, xacro)
@@ -145,5 +145,5 @@
         <!-- <origin xyz="0.27 0.21 0.7" rpy="0 0.65 -0.16" /> -->
         <!-- New values -->
-        <origin xyz="0.285 0.21 0.77" rpy="0.0 0.64 -0.14" />
+        <origin xyz="0.27 0.21 0.7" rpy="0.0 0.64 -0.14" />
         <parent link="base_footprint" />
         <child link="camera_link" />

Commit message: Added documentation and media, cleaned code

File: src/lx_autonomy/src/lx_packages/lx_description/urdf/lunarx.urdf.xacro (robot description, xacro)
@@ -142,7 +142,4 @@
     <link name="camera_link"/>
     <joint type="fixed" name="camera_link_joint">
-        <!-- old values  -->
-        <!-- <origin xyz="0.27 0.21 0.7" rpy="0 0.65 -0.16" /> -->
-        <!-- New values -->
         <origin xyz="0.27 0.21 0.7" rpy="0.0 0.64 -0.14" />
         <parent link="base_footprint" />
